File: schematics/z80-schematics.sch (KiCad schematic (older format))
At the start: 6 parts

Commit message: Non-I/O digital logic complete - CPU, ROM, RAM, bank switching and glue
Parts:
- added R? (x8): R, ~, symbol R
- added U?: 74LS540, ~, symbol 74LS540
- added U? (x2): 74LS289, ~, symbol 74LS289
- added U? (x3): 7400, ~, symbol 7400
- added U? (x2): 74LS32, ~, symbol 74LS32
Connections:
- net labels added: /banken, /banksel, /bankwr, /iorq, /mreq, /rd, /reset, /wr, a[12..15], b17, b18, b19, b[12..19]
- net labels removed: b[12..15], iorq, rd
- wire segments 113 -> 222
Other:
- moved on the sheet: U?

Commit message: Moving main buses over to label-based connections for improved readability
Connections:
- net labels removed: a[0..11], a[12..15], b[12..19], d[0..7]
- wire segments 222 -> 240

Commit message: Tidied up the bank-switcher (changed to label-based connections)
Connections:
- wire segments 240 -> 220
Other:
- moved on the sheet: U?, U?B, U?C

Commit message: Further label-ification
Connections:
- wire segments 220 -> 203
Changed lines of the file:
@@
 L VCC #PWR?
 U 1 1 5435B495
-P 6400 2950
-F 0 "#PWR?" H 6400 3050 30  0001 C CNN
-F 1 "VCC" H 6400 3050 30  0000 C CNN
-F 2 "" H 6400 2950 60  0000 C CNN
-F 3 "" H 6400 2950 60  0000 C CNN
-	1    6400 2950
+P 6200 2950
+F 0 "#PWR?" H 6200 3050 30  0001 C CNN
+F 1 "VCC" H 6200 3050 30  0000 C CNN
+F 2 "" H 6200 2950 60  0000 C CNN
+F 3 "" H 6200 2950 60  0000 C CNN
+	1    6200 2950
 	1    0    0    -1
 $EndComp
@@
 Text Label 8650 3350 2    60   Italic 12
 a15
-Text Label 6850 4750 0    60   Italic 12
+Text Label 3550 3850 0    60   Italic 12
 /rd
 $Comp
@@
 Text Label 6200 2150 0    60   Italic 12
 /iorq
-Text Label 6850 750  0    60   Italic 12
+Text Label 6150 3450 0    60   Italic 12
 /reset
-Text Label 6850 1150 0    60   Italic 12
+Text Label 6200 2250 0    60   Italic 12
 /wr
 Text Label 9200 2450 0    60   Italic 12
@@
 	3750 3850 3550 3850
 Wire Wire Line
-	6550 3650 6400 3650
-Wire Wire Line
-	6400 3650 6400 2950
-Wire Wire Line
-	6400 2950 6550 2950
+	6550 3650 6200 3650
+Wire Wire Line
+	6200 2950 6550 2950
 Wire Wire Line
 	6550 3450 6150 3450
 Wire Wire Line
-	6150 750  6150 3450
-Wire Wire Line
-	6150 3450 6150 5750
-Wire Wire Line
 	6550 3150 5950 3150
 Wire Wire Line
 	5950 3150 5950 5750
 Wire Wire Line
-	6550 2050 5700 2050
-Wire Wire Line
-	5700 2050 5700 4950
+	6550 2050 6200 2050
 Wire Wire Line
 	6550 1850 5600 1850
@@
 	3450 3750 3450 5150
 Wire Wire Line
-	3750 3650 3350 3650
-Wire Wire Line
-	3350 3650 3350 4950
+	3750 3650 3400 3650
 Wire Wire Line
 	8450 3050 8650 3050
@@
 	12200 3450 11750 3450
 Wire Wire Line
-	3550 3850 3550 4750
-Wire Wire Line
-	6150 750  9550 750
-Connection ~ 6150 3450
-Wire Wire Line
 	12650 3850 13100 3850
 Wire Wire Line
-	3100 1150 6450 1150
-Wire Wire Line
-	6450 1150 9250 1150
-Wire Wire Line
-	6550 2250 6450 2250
-Wire Wire Line
-	6450 2250 6450 1150
-Wire Wire Line
-	6550 2350 5800 2350
-Wire Wire Line
-	1100 4750 3550 4750
-Wire Wire Line
-	3550 4750 5800 4750
-Wire Wire Line
-	5800 4750 8300 4750
+	6550 2250 6200 2250
+Wire Wire Line
+	6550 2350 6200 2350
 Wire Wire Line
 	10750 2450 11200 2450
@@
 	10750 1850 11200 1850
 Wire Wire Line
-	5800 2350 5800 4750
-Wire Wire Line
-	1100 4750 1100 3550
-Wire Wire Line
-	1100 3550 1200 3550
-Connection ~ 5800 4750
-Connection ~ 3550 4750
-Wire Wire Line
-	3100 1150 3100 3950
-Connection ~ 6450 1150
+	1000 3550 1200 3550
 Connection ~ 14400 3950
 Wire Wire Line
@@
 	1200 5050 1250 5050
 Wire Wire Line
-	5700 4950 3350 4950
-Wire Wire Line
 	3350 4950 2450 4950
-Connection ~ 3350 4950
-Text Label 3550 4950 0    60   Italic 12
+Text Label 2650 4950 0    60   Italic 12
 /mreq
 $Comp
@@
 Text Label 12650 3850 0    60   Italic 12
 /reset
+Text Label 3100 3950 0    60   Italic 12
+/wr
+Text Label 1000 3550 0    60   Italic 12
+/rd
+Text Label 6200 2350 0    60   Italic 12
+/rd
+Text Label 3400 3650 0    60   Italic 12
+/mreq
+Text Label 6200 2050 0    60   Italic 12
+/mreq
+$Comp
+L VCC #PWR?
+U 1 1 5439C872
+P 6200 3650
+F 0 "#PWR?" H 6200 3750 30  0001 C CNN
+F 1 "VCC" H 6200 3750 30  0000 C CNN
+F 2 "" H 6200 3650 60  0000 C CNN
+F 3 "" H 6200 3650 60  0000 C CNN
+	1    6200 3650
+	1    0    0    -1
+$EndComp
 $EndSCHEMATC

Commit message: Finished switching to label-based connections
Connections:
- net labels added: /b19, /rom
- wire segments 203 -> 200
Other:
- moved on the sheet: U?, U?A

Commit message: Added odds and ends to the schematic
Parts:
- added C? (x2): C, symbol C
- added D?: LED, symbol LED
- added R? (x3): R, symbol R
- added SW? (x2): SW_PUSH, symbol SW_PUSH
- added X?: XO-14S, symbol XO-14S
Connections:
- net labels added: /nmi, GND, clk
- wire segments 200 -> 221
- no-connect marks 3 -> 4

Commit message: Marked resistors as 10k
Parts:
- R? (x11): value R -> 10k
Changed lines of the file:
@@
 P 14850 2450
 F 0 "R?" V 14930 2450 40  0000 C CNN
-F 1 "R" V 14857 2451 40  0000 C CNN
+F 1 "10k" V 14857 2451 40  0000 C CNN
 F 2 "~" V 14780 2450 30  0000 C CNN
 F 3 "~" H 14850 2450 30  0000 C CNN
@@
 P 14850 2600
 F 0 "R?" V 14930 2600 40  0000 C CNN
-F 1 "R" V 14857 2601 40  0000 C CNN
+F 1 "10k" V 14857 2601 40  0000 C CNN
 F 2 "~" V 14780 2600 30  0000 C CNN
 F 3 "~" H 14850 2600 30  0000 C CNN
@@
 P 14850 2750
 F 0 "R?" V 14930 2750 40  0000 C CNN
-F 1 "R" V 14857 2751 40  0000 C CNN
+F 1 "10k" V 14857 2751 40  0000 C CNN
 F 2 "~" V 14780 2750 30  0000 C CNN
 F 3 "~" H 14850 2750 30  0000 C CNN
@@
 P 14850 2900
 F 0 "R?" V 14930 2900 40  0000 C CNN
-F 1 "R" V 14857 2901 40  0000 C CNN
+F 1 "10k" V 14857 2901 40  0000 C CNN
 F 2 "~" V 14780 2900 30  0000 C CNN
 F 3 "~" H 14850 2900 30  0000 C CNN
@@
 P 14850 3050
 F 0 "R?" V 14930 3050 40  0000 C CNN
-F 1 "R" V 14857 3051 40  0000 C CNN
+F 1 "10k" V 14857 3051 40  0000 C CNN
 F 2 "~" V 14780 3050 30  0000 C CNN
 F 3 "~" H 14850 3050 30  0000 C CNN
@@
 P 14850 3200
 F 0 "R?" V 14930 3200 40  0000 C CNN
-F 1 "R" V 14857 3201 40  0000 C CNN
+F 1 "10k" V 14857 3201 40  0000 C CNN
 F 2 "~" V 14780 3200 30  0000 C CNN
 F 3 "~" H 14850 3200 30  0000 C CNN
@@
 P 14850 3350
 F 0 "R?" V 14930 3350 40  0000 C CNN
-F 1 "R" V 14857 3351 40  0000 C CNN
+F 1 "10k" V 14857 3351 40  0000 C CNN
 F 2 "~" V 14780 3350 30  0000 C CNN
 F 3 "~" H 14850 3350 30  0000 C CNN
@@
 P 14850 3500
 F 0 "R?" V 14930 3500 40  0000 C CNN
-F 1 "R" V 14857 3501 40  0000 C CNN
+F 1 "10k" V 14857 3501 40  0000 C CNN
 F 2 "~" V 14780 3500 30  0000 C CNN
 F 3 "~" H 14850 3500 30  0000 C CNN
@@
 P 1000 5500
 F 0 "R?" V 1080 5500 40  0000 C CNN
-F 1 "R" V 1007 5501 40  0000 C CNN
+F 1 "10k" V 1007 5501 40  0000 C CNN
 F 2 "" V 930 5500 30  0000 C CNN
 F 3 "" H 1000 5500 30  0000 C CNN
@@
 P 1550 4650
 F 0 "R?" V 1630 4650 40  0000 C CNN
-F 1 "R" V 1557 4651 40  0000 C CNN
+F 1 "10k" V 1557 4651 40  0000 C CNN
 F 2 "" V 1480 4650 30  0000 C CNN
 F 3 "" H 1550 4650 30  0000 C CNN
@@
 P 2250 4650
 F 0 "R?" V 2330 4650 40  0000 C CNN
-F 1 "R" V 2257 4651 40  0000 C CNN
+F 1 "10k" V 2257 4651 40  0000 C CNN
 F 2 "" V 2180 4650 30  0000 C CNN
 F 3 "" H 2250 4650 30  0000 C CNN

Commit message: Added the CTC wiring
Parts:
- added R?: R, symbol R
Connections:
- net labels added: /ctcsel, /int, /m1, ieo, to0, to1, to2
- wire segments 221 -> 263
- no-connect marks 4 -> 7
Other:
- moved on the sheet: U?
