File: schematics/z80-schematics.kicad_sch (KiCad schematic)
At the start: 56 parts, among them P1 FTDI SERIAL, P2 CONN_02X08, P3 CONN_01X06, SW1 SW_PUSH, SW2 SW_PUSH, U1 Z80-CPU, U10 Z80-CTC, U11 Z80-SIO/0, U12 74HC574, U13 74HC541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

Commit message: Switch other standard parts to standard library parts
Parts:
- P2: symbol z80-schematics-rescue:CONN_02X08 -> Connector_Generic:Conn_02x08_Odd_Even
- U12: symbol z80-schematics-rescue:74LS574 -> 74xx:74LS574
- U13: symbol z80-schematics-rescue:74LS541 -> 74xx:74LS541
- U2: symbol z80-schematics-rescue:628128 -> Memory_RAM:628128_DIP32_SSOP32
- U3: symbol z80-schematics-rescue:28C256-RESCUE-z80-schematics -> Memory_EEPROM:28C256
- U6: symbol z80-schematics-rescue:74LS138 -> 74xx:74LS138
- U7: symbol z80-schematics-rescue:74LS540 -> 74xx:74LS540
- U8: symbol z80-schematics-rescue:7400 -> 74xx:7400
- U9: symbol z80-schematics-rescue:74LS32 -> 74xx:74LS32
Connections:
- net +5V: no longer U8.14 (VCC), U8.14 (VCC), U8.14 (VCC), U8.14 (VCC), U9.14 (VCC), U9.14 (VCC), U9.14 (VCC), U9.14 (VCC)
- net GND: no longer U8.7 (GND), U8.7 (GND), U8.7 (GND), U8.7 (GND), U9.7 (GND), U9.7 (GND), U9.7 (GND), U9.7 (GND)
Other:
- moved on the sheet: R1, R2, R3, R4, R5, R6, R7, R8

Commit message: Rename the rescue library to no longer be a rescue library.
Parts:
- U1: symbol z80-schematics-rescue:Z80-CPU -> z80-schematics:Z80-CPU
- U10: symbol z80-schematics-rescue:Z80-CTC -> z80-schematics:Z80-CTC
- U11: symbol z80-schematics-rescue:Z80-SIO/0 -> z80-schematics:Z80-SIO/0
- U4, U5: symbol z80-schematics-rescue:74LS289 -> z80-schematics:74LS289
Changed lines of the file:
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@@
     )
   )
-  (symbol (lib_id "z80-schematics-rescue:Z80-CPU") (at 193.04 52.07 0) (unit 1)
+  (symbol (lib_id "z80-schematics:Z80-CPU") (at 193.04 52.07 0) (unit 1)
     (in_bom yes) (on_board yes) (dnp no)
     (property "Reference" "U1" (at 193.04 17.78 0)
@@
     )
   )
-  (symbol (lib_id "z80-schematics-rescue:Z80-CTC") (at 193.04 125.73 0) (unit 1)
+  (symbol (lib_id "z80-schematics:Z80-CTC") (at 193.04 125.73 0) (unit 1)
     (in_bom yes) (on_board yes) (dnp no)
     (property "Reference" "U10" (at 193.04 97.79 0)
@@
     )
   )
-  (symbol (lib_id "z80-schematics-rescue:Z80-SIO/0") (at 260.35 127 0) (unit 1)
+  (symbol (lib_id "z80-schematics:Z80-SIO/0") (at 260.35 127 0) (unit 1)
     (in_bom yes) (on_board yes) (dnp no)
     (property "Reference" "U11" (at 260.35 96.52 0)
@@
     )
   )
-  (symbol (lib_id "z80-schematics-rescue:74LS289") (at 327.66 34.29 0) (unit 1)
+  (symbol (lib_id "z80-schematics:74LS289") (at 327.66 34.29 0) (unit 1)
     (in_bom yes) (on_board yes) (dnp no)
     (property "Reference" "U4" (at 332.74 19.05 0)
@@
     )
   )
-  (symbol (lib_id "z80-schematics-rescue:74LS289") (at 378.46 33.02 0) (unit 1)
+  (symbol (lib_id "z80-schematics:74LS289") (at 378.46 33.02 0) (unit 1)
     (in_bom yes) (on_board yes) (dnp no)
     (property "Reference" "U5" (at 383.54 17.78 0)

Commit message: Fix DRC error (missing power units on the updated 74xx chips).
Parts:
- added unit 5 of U8
- added unit 5 of U9
Connections:
- net +5V: now also U8.14 (VCC), U9.14 (VCC)
- net GND: now also U8.7 (GND), U9.7 (GND)
Changed lines of the file:
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@@
+    )
+  )
+  (symbol (lib_id "74xx:74LS32") (at 54.61 228.6 0) (unit 5)
+    (in_bom yes) (on_board yes) (dnp no)
+    (property "Reference" "U9" (at 54.61 227.33 0)
+      (effects (font (size 1.524 1.524)))
+    )
+    (property "Value" "74HCT32" (at 54.61 229.87 0)
+      (effects (font (size 1.524 1.524)))
+    )
+    (property "Footprint" "~" (at 54.61 228.6 0)
+      (effects (font (size 1.27 1.27)) hide)
+    )
+    (property "Datasheet" "http://www.ti.com/lit/gpn/sn74LS32" (at 54.61 228.6 0)
+      (effects (font (size 1.27 1.27)) hide)
+    )
+    (pin "1")
+    (pin "2")
+    (pin "3")
+    (pin "4")
+    (pin "5")
+    (pin "6")
+    (pin "10")
+    (pin "8")
+    (pin "9")
+    (pin "11")
+    (pin "12")
+    (pin "13")
+    (pin "14")
+    (pin "7")
+    (instances
+      (project "z80-schematics"
+        (path "/2c0e1a0c-15a7-4cf5-99de-7d26825760fb"
+          (reference "U9") (unit 5)
+        )
+      )
+    )
+  )
+  (symbol (lib_id "power:GND") (at 54.61 241.3 0) (unit 1)
+    (in_bom yes) (on_board yes) (dnp no)
+    (property "Reference" "#PWR051" (at 54.61 241.3 0)
+      (effects (font (size 0.762 0.762)) hide)
+    )
+    (property "Value" "GND" (at 54.61 243.078 0)
+      (effects (font (size 0.762 0.762)) hide)
+    )
+    (property "Footprint" "" (at 54.61 241.3 0)
+      (effects (font (size 1.27 1.27)) hide)
+    )
+    (property "Datasheet" "" (at 54.61 241.3 0)
+      (effects (font (size 1.27 1.27)) hide)
+    )
+    (pin "1")
+    (instances
+      (project "z80-schematics"
+        (path "/2c0e1a0c-15a7-4cf5-99de-7d26825760fb"
+          (reference "#PWR051") (unit 1)
+        )
+      )
+    )
+  )
+  (symbol (lib_id "power:VCC") (at 41.91 215.9 0) (unit 1)
+    (in_bom yes) (on_board yes) (dnp no)
+    (property "Reference" "#PWR048" (at 41.91 213.36 0)
+      (effects (font (size 0.762 0.762)) hide)
+    )
+    (property "Value" "VCC" (at 41.91 213.36 0)
+      (effects (font (size 0.762 0.762)))
+    )
+    (property "Footprint" "" (at 41.91 215.9 0)
+      (effects (font (size 1.27 1.27)) hide)
+    )
+    (property "Datasheet" "" (at 41.91 215.9 0)
+      (effects (font (size 1.27 1.27)) hide)
+    )
+    (pin "1")
+    (instances
+      (project "z80-schematics"
+        (path "/2c0e1a0c-15a7-4cf5-99de-7d26825760fb"
+          (reference "#PWR048") (unit 1)
+        )
+      )
     )
   )
@@
     )
   )
+  (symbol (lib_id "power:VCC") (at 54.61 215.9 0) (unit 1)
+    (in_bom yes) (on_board yes) (dnp no)
+    (property "Reference" "#PWR049" (at 54.61 213.36 0)
+      (effects (font (size 0.762 0.762)) hide)
+    )
+    (property "Value" "VCC" (at 54.61 213.36 0)
+      (effects (font (size 0.762 0.762)))
+    )
+    (property "Footprint" "" (at 54.61 215.9 0)
+      (effects (font (size 1.27 1.27)) hide)
+    )
+    (property "Datasheet" "" (at 54.61 215.9 0)
+      (effects (font (size 1.27 1.27)) hide)
+    )
+    (pin "1")
+    (instances
+      (project "z80-schematics"
+        (path "/2c0e1a0c-15a7-4cf5-99de-7d26825760fb"
+          (reference "#PWR049") (unit 1)
+        )
+      )
+    )
+  )
   (symbol (lib_id "power:GND") (at 326.39 102.87 0) (unit 1)
     (in_bom yes) (on_board yes) (dnp no)
@@
     )
   )
+  (symbol (lib_id "power:GND") (at 41.91 241.3 0) (unit 1)
+    (in_bom yes) (on_board yes) (dnp no)
+    (property "Reference" "#PWR050" (at 41.91 241.3 0)
+      (effects (font (size 0.762 0.762)) hide)
+    )
+    (property "Value" "GND" (at 41.91 243.078 0)
+      (effects (font (size 0.762 0.762)) hide)
+    )
+    (property "Footprint" "" (at 41.91 241.3 0)
+      (effects (font (size 1.27 1.27)) hide)
+    )
+    (property "Datasheet" "" (at 41.91 241.3 0)
+      (effects (font (size 1.27 1.27)) hide)
+    )
+    (pin "1")
+    (instances
+      (project "z80-schematics"
+        (path "/2c0e1a0c-15a7-4cf5-99de-7d26825760fb"
+          (reference "#PWR050") (unit 1)
+        )
+      )
+    )
+  )
   (symbol (lib_id "power:GND") (at 256.54 69.85 0) (unit 1)
     (in_bom yes) (on_board yes) (dnp no)
@@
         )
       )
+    )
+  )
+  (symbol (lib_id "74xx:7400") (at 41.91 228.6 0) (unit 5)
+    (in_bom yes) (on_board yes) (dnp no)
+    (property "Reference" "U8" (at 41.91 227.33 0)
+      (effects (font (size 1.524 1.524)))
+    )
+    (property "Value" "74HCT00" (at 41.91 231.14 0)
+      (effects (font (size 1.524 1.524)))
+    )
+    (property "Footprint" "~" (at 41.91 228.6 0)
+      (effects (font (size 1.27 1.27)) hide)
+    )
+    (property "Datasheet" "http://www.ti.com/lit/gpn/sn7400" (at 41.91 228.6 0)
+      (effects (font (size 1.27 1.27)) hide)
+    )
+    (pin "1")
+    (pin "2")
+    (pin "3")
+    (pin "4")
+    (pin "5")
+    (pin "6")
+    (pin "10")
+    (pin "8")
+    (pin "9")
+    (pin "11")
+    (pin "12")
+    (pin "13")
+    (pin "14")
+    (pin "7")
+    (instances
+      (project "z80-schematics"
+        (path "/2c0e1a0c-15a7-4cf5-99de-7d26825760fb"
+          (reference "U8") (unit 5)
+        )
+      )
